File: 2025SIMPLETVC.kicad_pcb (KiCad board)
At the start: 4 copper layers, 55 x 140 mm, 41 parts, among them J10 BATT, J2 SRV 1, J3 SRV 2, J4 ELEC ARM, J5 PYRO ARM, J6 PYRO 1, J7 UART1 5V, J8 PYRO 2, Q1 BSS138, Q2 BSS138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

Commit message: v1.0 finished
Parts:
- C19, C2, C22: footprint Capacitor_SMD:C_0402_1005Metric -> Capacitor_SMD:C_0603_1608Metric
- moved C2 0.60 mm to (153.7, 150.3)
- moved C22 0.42 mm to (156.8, 131.1)
- moved C1 0.30 mm to (156.2, 145.8)
